File: ws-control-board/ws-control-board/ws-control-board.kicad_pcb (KiCad board)
At the start: 2 copper layers, 84.5 x 68.6 mm, 15 parts, among them J1 Conn_01x15_Socket, J2 Conn_01x15_Socket, J3 Conn_01x07_Socket, J4 Conn_01x06_Socket, J5 Conn_01x06_Socket, J6 Screw_Terminal_01x03, J7 Screw_Terminal_01x02, J8 Screw_Terminal_01x02

Commit message: Fix board bugs
Connections:
- J2 pad 11: /PHOTO_SENS -> unconnected-(J2-Pin_11-Pad11)
- J2 pad 15: VIN -> unconnected-(J2-Pin_15-Pad15)
- J2 pad 6: unconnected-(J2-Pin_6-Pad6) -> /PHOTO_SENS
- J8 pad 1: VIN -> +3.3V
Routing:
- net +3.3V: track 159.9 -> 178.6 mm
- net VIN: track 18.2 -> 0.00 mm
- net /PHOTO_SENS: track 24.3 -> 15.5 mm
Changed lines of the file:
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@@
 	(net 20 "unconnected-(J2-Pin_1-Pad1)")
 	(net 21 "/PHOTO_SENS")
-	(net 22 "unconnected-(J2-Pin_6-Pad6)")
+	(net 22 "unconnected-(J2-Pin_11-Pad11)")
 	(net 23 "unconnected-(J2-Pin_10-Pad10)")
 	(net 24 "unconnected-(J2-Pin_13-Pad13)")
@@
 	(net 28 "unconnected-(J2-Pin_3-Pad3)")
 	(net 29 "unconnected-(J2-Pin_8-Pad8)")
-	(net 30 "VIN")
+	(net 30 "unconnected-(J2-Pin_15-Pad15)")
 	(net 31 "unconnected-(J3-Pin_5-Pad5)")
 	(net 32 "unconnected-(J4-Pin_2-Pad2)")
@@
 			(net 14 "unconnected-(J1-Pin_5-Pad5)")
 			(pinfunction "Pin_5")
-			(pintype "passive")
+			(pintype "passive+no_connect")
 		)
 		(pad "6" thru_hole oval
@@
 			(net 9 "unconnected-(J1-Pin_11-Pad11)")
 			(pinfunction "Pin_11")
-			(pintype "passive")
+			(pintype "passive+no_connect")
 		)
 		(pad "12" thru_hole oval
@@
 			(net 6 "unconnected-(J1-Pin_12-Pad12)")
 			(pinfunction "Pin_12")
-			(pintype "passive")
+			(pintype "passive+no_connect")
 		)
 		(pad "13" thru_hole oval
@@
 			(net 13 "unconnected-(J1-Pin_13-Pad13)")
 			(pinfunction "Pin_13")
-			(pintype "passive")
+			(pintype "passive+no_connect")
 		)
 		(pad "14" thru_hole oval
@@
 			(layers "*.Cu" "*.Mask")
 			(remove_unused_layers no)
-			(net 30 "VIN")
+			(net 12 "+3.3V")
 			(pinfunction "Pin_1")
 			(pintype "passive")
@@
 			(net 20 "unconnected-(J2-Pin_1-Pad1)")
 			(pinfunction "Pin_1")
-			(pintype "passive")
+			(pintype "passive+no_connect")
 		)
 		(pad "2" thru_hole oval
@@
 			(net 27 "unconnected-(J2-Pin_2-Pad2)")
 			(pinfunction "Pin_2")
-			(pintype "passive")
+			(pintype "passive+no_connect")
 		)
 		(pad "3" thru_hole oval
@@
 			(net 28 "unconnected-(J2-Pin_3-Pad3)")
 			(pinfunction "Pin_3")
-			(pintype "passive")
+			(pintype "passive+no_connect")
 		)
 		(pad "4" thru_hole oval
@@
 			(net 19 "unconnected-(J2-Pin_4-Pad4)")
 			(pinfunction "Pin_4")
-			(pintype "passive")
+			(pintype "passive+no_connect")
 		)
 		(pad "5" thru_hole oval
@@
 			(layers "*.Cu" "*.Mask")
 			(remove_unused_layers no)
-			(net 22 "unconnected-(J2-Pin_6-Pad6)")
+			(net 21 "/PHOTO_SENS")
 			(pinfunction "Pin_6")
 			(pintype "passive")
@@
 			(net 25 "unconnected-(J2-Pin_7-Pad7)")
 			(pinfunction "Pin_7")
-			(pintype "passive")
+			(pintype "passive+no_connect")
 		)
 		(pad "8" thru_hole oval
@@
 			(net 29 "unconnected-(J2-Pin_8-Pad8)")
 			(pinfunction "Pin_8")
-			(pintype "passive")
+			(pintype "passive+no_connect")
 		)
 		(pad "9" thru_hole oval
@@
 			(net 18 "unconnected-(J2-Pin_9-Pad9)")
 			(pinfunction "Pin_9")
-			(pintype "passive")
+			(pintype "passive+no_connect")
 		)
 		(pad "10" thru_hole oval
@@
 			(net 23 "unconnected-(J2-Pin_10-Pad10)")
 			(pinfunction "Pin_10")
-			(pintype "passive")
+			(pintype "passive+no_connect")
 		)
 		(pad "11" thru_hole oval
@@
 			(layers "*.Cu" "*.Mask")
 			(remove_unused_layers no)
-			(net 21 "/PHOTO_SENS")
+			(net 22 "unconnected-(J2-Pin_11-Pad11)")
 			(pinfunction "Pin_11")
-			(pintype "passive")
+			(pintype "passive+no_connect")
 		)
 		(pad "12" thru_hole oval
@@
 			(net 24 "unconnected-(J2-Pin_13-Pad13)")
 			(pinfunction "Pin_13")
-			(pintype "passive")
+			(pintype "passive+no_connect")
 		)
 		(pad "14" thru_hole oval
@@
 			(layers "*.Cu" "*.Mask")
 			(remove_unused_layers no)
-			(net 30 "VIN")
+			(net 30 "unconnected-(J2-Pin_15-Pad15)")
 			(pinfunction "Pin_15")
-			(pintype "passive")
+			(pintype "passive+no_connect")
 		)
 		(embedded_fonts no)
@@
 		)
 	)
-	(gr_text "VIN"
+	(gr_text "3V3"
 		(at 108.585 112.776 0)
 		(layer "F.SilkS")
@@
 			(font
 				(size 1 1)
-				(thickness 0.127)
+				(thickness 0.15)
 			)
 			(justify bottom)
@@
 			(font
 				(size 1 1)
-				(thickness 0.127)
+				(thickness 0.15)
 			)
 			(justify left bottom)
@@
 			(font
 				(size 1 1)
-				(thickness 0.127)
+				(thickness 0.15)
 			)
 			(justify left bottom)
@@
 			(font
 				(size 1 1)
-				(thickness 0.127)
+				(thickness 0.15)
 			)
 			(justify left bottom)
@@
 			(font
 				(size 1 1)
-				(thickness 0.127)
+				(thickness 0.15)
 			)
 			(justify bottom)
@@
 			(font
 				(size 1 1)
-				(thickness 0.127)
+				(thickness 0.15)
 			)
 			(justify left bottom)
@@
 			(keep_text_aligned yes)
 		)
-		(gr_text "2.7"
+		(gr_text "68.58"
 			(at 94.735 90.17 90)
 			(layer "User.1")
@@
 			(keep_text_aligned yes)
 		)
-		(gr_text "2.9"
+		(gr_text "73.66"
 			(at 146.685 129.66 0)
 			(layer "User.1")
@@
 			(keep_text_aligned yes)
 		)
-		(gr_text "1.75"
+		(gr_text "44.45"
 			(at 191.255 98.044 90)
 			(layer "User.1")
@@
 			(keep_text_aligned yes)
 		)
-		(gr_text "3.325"
+		(gr_text "84.455"
 			(at 145.7325 48.38 0)
 			(layer "User.1")
@@
 			(keep_text_aligned yes)
 		)
-		(gr_text "2.4"
+		(gr_text "60.96"
 			(at 98.672 89.789 90)
 			(layer "User.1")
@@
 		(start 145.288 68.326)
 		(end 145.288 72.136)
-		(width 0.2)
+		(width 0.381)
 		(layer "F.Cu")
 		(net 8)
@@
 		(start 143.51 66.548)
 		(end 145.288 68.326)
-		(width 0.2)
+		(width 0.381)
 		(layer "F.Cu")
 		(net 8)
@@
 		(start 141.732 75.692)
 		(end 141.732 96.012)
-		(width 0.2)
+		(width 0.381)
 		(layer "F.Cu")
 		(net 8)
@@
 		(start 145.288 72.136)
 		(end 141.732 75.692)
-		(width 0.2)
+		(width 0.381)
 		(layer "F.Cu")
 		(net 8)
@@
 		(start 106.68 78.232)
 		(end 118.364 66.548)
-		(width 0.2)
+		(width 0.381)
 		(layer "F.Cu")
 		(net 8)
@@
 		(start 141.732 96.012)
 		(end 147.32 101.6)
-		(width 0.2)
+		(width 0.381)
 		(layer "F.Cu")
 		(net 8)
@@
 		(start 118.364 66.548)
 		(end 143.51 66.548)
-		(width 0.2)
+		(width 0.381)
 		(layer "F.Cu")
 		(net 8)
@@
 	)
 	(segment
+		(start 105.248 96.047)
+		(end 105.248 110.709)
+		(width 0.762)
+		(layer "F.Cu")
+		(net 12)
+	)
+	(segment
+		(start 105.248 110.709)
+		(end 106.68 112.141)
+		(width 0.762)
+		(layer "F.Cu")
+		(net 12)
+	)
+	(segment
 		(start 130.175 71.12)
 		(end 130.175 71.06)
@@
 	)
 	(segment
+		(start 106.68 94.615)
+		(end 105.248 96.047)
+		(width 0.762)
+		(layer "F.Cu")
+		(net 12)
+	)
+	(segment
 		(start 117.475 83.82)
 		(end 117.475 90.805)
@@
 	(segment
 		(start 116.84 97.155)
-		(end 106.68 97.155)
+		(end 121.285 97.155)
 		(width 0.381)
 		(layer "F.Cu")
@@
 	)
 	(segment
-		(start 121.92 109.22)
-		(end 116.84 104.14)
+		(start 116.84 97.155)
+		(end 106.68 97.155)
 		(width 0.381)
 		(layer "F.Cu")
@@
 	)
 	(segment
-		(start 116.84 104.14)
-		(end 116.84 97.155)
+		(start 121.285 97.155)
+		(end 121.92 96.52)
 		(width 0.381)
 		(layer "F.Cu")
@@
 		(net 26)
 	)
-	(segment
-		(start 109.601 112.141)
-		(end 116.84 119.38)
-		(width 0.762)
-		(layer "F.Cu")
-		(net 30)
-	)
-	(segment
-		(start 116.84 119.38)
-		(end 121.92 119.38)
-		(width 0.762)
-		(layer "F.Cu")
-		(net 30)
-	)
-	(segment
-		(start 106.68 112.141)
-		(end 109.601 112.141)
-		(width 0.762)
-		(layer "F.Cu")
-		(net 30)
-	)
 	(zone
