File: ws-control-board/ws-control-board/ws-control-board.kicad_sch (KiCad schematic)
At the start: 15 parts, among them J1 Conn_01x15_Socket, J2 Conn_01x15_Socket, J3 Conn_01x07_Socket, J4 Conn_01x06_Socket, J5 Conn_01x06_Socket, J6 Screw_Terminal_01x03, J7 Screw_Terminal_01x02, J8 Screw_Terminal_01x02

Commit message: Fix board bugs
Connections:
- net +3.3V: now also J8.1 (Pin_1)
- net PHOTO_SENS: now also J2.6 (Pin_6); no longer J2.11 (Pin_11)
- net VIN: no longer names the net of J2.15 (Pin_15)
- net VIN: no longer J8.1 (Pin_1)
- no-connect marks 5 -> 20
Changed lines of the file:
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@@
 		)
 	)
-	(text_box "Bradley University ECE Department SPR 2025 ECE 398\nWeather Station Group\n\nCarrier board for off-the-shelf breakout boards which will be used \ninside of the weather staiton enclosure. This includes the microcontroller\nand all necessary peripherals to operate the weather station.\n\nIn the future, this board should just include all necessary components\nrather than breakout boards. \n\nTODO: \n- [ ] Check that board is mechanically\n          spaced properly (all boards contained in silk,\n          pins properly seperated, we have connectors for .1in\n          pitch footprint, a terminal block will fit)\n- [ ] Pinout is correct when plugged into board\n- [ ] Spacing of ESP header is correct\n- [ ] Sunny buddy would work with this\n\nLast Revision: Jacob Simeone 2025-03-28"
+	(text_box "Bradley University ECE Department SPR 2025 ECE 398\nWeather Station Group\n\nCarrier board for off-the-shelf breakout boards which will be used \ninside of the weather staiton enclosure. This includes the microcontroller\nand all necessary peripherals to operate the weather station.\n\nIn the future, this board should just include all necessary components\nrather than breakout boards. \n\nTODO: \n- [X] Check that board is mechanically\n          spaced properly (all boards contained in silk,\n          pins properly seperated, we have connectors for .1in\n          pitch footprint, a terminal block will fit)\n- [X] Pinout is correct when plugged into board\n- [X] Spacing of ESP header is correct\n- [ ] Break out unused controller connections\n- [ ] Silkscreen writing on stat codes\n- [ ] Sunny buddy would work with this\n\nLast Revision: Jacob Simeone 2025-03-28"
 		(exclude_from_sim no)
 		(at 16.51 19.05 0)
@@
 	)
 	(no_connect
+		(at 224.79 73.66)
+	)
+	(no_connect
 		(at 121.92 78.74)
+	)
+	(no_connect
+		(at 224.79 83.82)
 	)
 	(no_connect
@@
 	)
 	(no_connect
+		(at 257.81 99.06)
+	)
+	(no_connect
+		(at 257.81 93.98)
+	)
+	(no_connect
+		(at 224.79 76.2)
+	)
+	(no_connect
+		(at 224.79 86.36)
+	)
+	(no_connect
+		(at 224.79 91.44)
+	)
+	(no_connect
+		(at 224.79 99.06)
+	)
+	(no_connect
+		(at 224.79 93.98)
+	)
+	(no_connect
 		(at 257.81 73.66)
+	)
+	(no_connect
+		(at 224.79 68.58)
+	)
+	(no_connect
+		(at 224.79 104.14)
+	)
+	(no_connect
+		(at 224.79 88.9)
 	)
 	(no_connect
@@
 	)
 	(no_connect
+		(at 224.79 71.12)
+	)
+	(no_connect
+		(at 257.81 78.74)
+	)
+	(no_connect
 		(at 251.46 40.64)
 	)
+	(no_connect
+		(at 257.81 96.52)
+	)
 	(wire
 		(pts
@@
 	(wire
 		(pts
-			(xy 218.44 93.98) (xy 224.79 93.98)
+			(xy 218.44 81.28) (xy 224.79 81.28)
 		)
 		(stroke
@@
 	(wire
 		(pts
-			(xy 207.01 104.14) (xy 207.01 102.87)
-		)
-		(stroke
-			(width 0)
-			(type default)
-		)
-	)
-	(wire
-		(pts
 			(xy 257.81 71.12) (xy 262.89 71.12)
 		)
@@
 		(pts
 			(xy 158.75 71.12) (xy 162.56 71.12)
-		)
-		(stroke
-			(width 0)
-			(type default)
-		)
-	)
-	(wire
-		(pts
-			(xy 224.79 104.14) (xy 207.01 104.14)
 		)
 		(stroke
@@
 	)
 	(label "PHOTO_SENS"
-		(at 218.44 93.98 180)
+		(at 218.44 81.28 180)
 		(effects
 			(font
@@
 	)
 	(symbol
-		(lib_id "power:+3.3V")
-		(at 191.77 71.12 0)
-		(unit 1)
-		(exclude_from_sim no)
-		(in_bom yes)
-		(on_board yes)
-		(dnp no)
-		(fields_autoplaced yes)
-		(property "Reference" "#PWR017"
-			(at 191.77 74.93 0)
-			(effects
-				(font
-					(size 1.27 1.27)
-				)
-				(hide yes)
-			)
-		)
-		(property "Value" "VIN"
-			(at 191.77 66.04 0)
-			(effects
-				(font
-					(size 1.27 1.27)
-				)
-			)
-		)
-		(property "Footprint" ""
-			(at 191.77 71.12 0)
-			(effects
-				(font
-					(size 1.27 1.27)
-				)
-				(hide yes)
-			)
-		)
-		(property "Datasheet" ""
-			(at 191.77 71.12 0)
-			(effects
-				(font
-					(size 1.27 1.27)
-				)
-				(hide yes)
-			)
-		)
-		(property "Description" "Power symbol creates a global label with name \"+3.3V\""
-			(at 191.77 71.12 0)
-			(effects
-				(font
-					(size 1.27 1.27)
-				)
-				(hide yes)
-			)
-		)
-		(pin "1"
-		)
-		(instances
-			(project "ws-control-board"
-				(path "/76b5f725-792b-4832-8607-f92582a36140"
-					(reference "#PWR017")
-					(unit 1)
-				)
-			)
-		)
-	)
-	(symbol
 		(lib_id "Connector:Screw_Terminal_01x02")
 		(at 109.22 31.75 0)
@@
 	)
 	(symbol
-		(lib_id "power:VDD")
-		(at 207.01 102.87 0)
-		(unit 1)
-		(exclude_from_sim no)
-		(in_bom yes)
-		(on_board yes)
-		(dnp no)
-		(property "Reference" "#PWR014"
-			(at 207.01 106.68 0)
-			(effects
-				(font
-					(size 1.27 1.27)
-				)
-				(hide yes)
-			)
-		)
-		(property "Value" "VIN"
-			(at 207.01 99.06 0)
-			(effects
-				(font
-					(size 1.27 1.27)
-				)
-			)
-		)
-		(property "Footprint" ""
-			(at 207.01 102.87 0)
-			(effects
-				(font
-					(size 1.27 1.27)
-				)
-				(hide yes)
-			)
-		)
-		(property "Datasheet" ""
-			(at 207.01 102.87 0)
-			(effects
-				(font
-					(size 1.27 1.27)
-				)
-				(hide yes)
-			)
-		)
-		(property "Description" "Power symbol creates a global label with name \"VDD\""
-			(at 207.01 102.87 0)
-			(effects
-				(font
-					(size 1.27 1.27)
-				)
-				(hide yes)
-			)
-		)
-		(pin "1"
-		)
-		(instances
-			(project ""
-				(path "/76b5f725-792b-4832-8607-f92582a36140"
-					(reference "#PWR014")
-					(unit 1)
-				)
-			)
-		)
-	)
-	(symbol
 		(lib_id "Connector:Conn_01x15_Socket")
 		(at 252.73 86.36 0)
@@
 					(unit 1)
 				)
+			)
+		)
+	)
+	(symbol
+		(lib_id "power:+3.3V")
+		(at 191.77 71.12 0)
+		(unit 1)
+		(exclude_from_sim no)
+		(in_bom yes)
+		(on_board yes)
+		(dnp no)
+		(fields_autoplaced yes)
+		(property "Reference" "#PWR014"
+			(at 191.77 74.93 0)
+			(effects
+				(font
+					(size 1.27 1.27)
+				)
+				(hide yes)
+			)
+		)
+		(property "Value" "+3.3V"
+			(at 191.77 66.04 0)
+			(effects
+				(font
+					(size 1.27 1.27)
+				)
+			)
+		)
+		(property "Footprint" ""
+			(at 191.77 71.12 0)
+			(effects
+				(font
+					(size 1.27 1.27)
+				)
+				(hide yes)
+			)
+		)
+		(property "Datasheet" ""
+			(at 191.77 71.12 0)
+			(effects
+				(font
+					(size 1.27 1.27)
+				)
+				(hide yes)
+			)
+		)
+		(property "Description" "Power symbol creates a global label with name \"+3.3V\""
+			(at 191.77 71.12 0)
+			(effects
+				(font
+					(size 1.27 1.27)
+				)
+				(hide yes)
+			)
+		)
+		(pin "1"
+		)
+		(instances
+			(project "ws-control-board"
+				(path "/76b5f725-792b-4832-8607-f92582a36140"
+					(reference "#PWR014")
+					(unit 1)
+				)
